File: sensor_base.kicad_sch (KiCad schematic)
At the start: 28 parts, among them J14 Calibration_In, J2 PT-100_TEMP_IN, J5 SPARE, U11 OPA2397DGKR, U17 DHT20, U3 ESDA5V3SC5

Commit message: BUG_FIX ------- - Swapped ground for the 2.5V reference on the non-inverting leg of U11B (External temperature probe)   This is due to the fact that the temp probe voltage can go both above and below the reference point so we need something higher than ground to prevent pegging the output to 0 when temp probe impedance drops below 1k.
FEATURES
--------
- Finalized many of the parts for the BOM
Parts:
- C1, C2, C3: value C -> 800n
- R1, R50, R51: value R -> 1k
- R21, R9: value R -> 100k
- R42, R46: value R -> 10k
- R47, R7: value R -> 10
- R48, R49: value R -> 200
- R52: value 5k -> 1k
Connections:
- net ANALOG_GND: no longer R9.1
- new net +2.5V_REF: R9.1
Other:
- note added: "1k gives a an average current of ~2mA and Vsense of ~2V"
- note added: "Assuming 2Amp max; Vsense = 2*0.1 = 200mV Gain = 4.096V/200mV = ~20"
- note added: "Gain = 10"
- note added: "R42 and R46 should be matched. R21 and R9 should be matched."
- note removed: "5k gives a an average current of 0.7mA and Vsense of 683mV"
- note removed: "Gain = TODO"
- note removed: "R42 and R21 should be matched. R46 and R9 should be matched."
